File: PCB/sch/Baby_Mon_V0/baby_monitor_v0.brd (EAGLE design)
At the start: 20 x 20 mm, 37 parts, among them J1 BATT-COIN1CR1216, U1 NRF5340-QKAA-AB0-R, U2 MAX30101EFD+, U3 MAX30205MTA+, X1 XRCGB32M000F2P10R0

Commit message: u
Parts:
- added SW2: (no value), graftel-internal-ic:MICROBUILDER_BTN_EVQPQ_4.5MM
- added U$2: (no value), graftel-internal-ic:MICROBUILDER_APA102_2020
- moved C2 11.4 mm to (0.08, 14.0), turned to 180 degrees
- moved C3 10.6 mm to (-1.32, 9.77)
- moved C7 8.27 mm to (11.6, 12.8), turned to 0 degrees
- moved C1 7.63 mm to (0.32, 9.92), turned to 180 degrees
- moved C12 6.87 mm to (5.61, 0.97), flipped to the top, turned to 0 degrees
- moved C13 3.94 mm to (7.30, 3.02), flipped to the top, turned to 90 degrees
- moved C11 2.75 mm to (-0.42, 3.69), flipped to the bottom, turned to 90 degrees
- moved J8 2.35 mm to (13.7, 5.77)
- moved J7 2.27 mm to (14.2, 7.37)
- moved C4 2.27 mm to (11.6, 10.5)
- moved C5 2.27 mm to (11.6, 9.31)
- moved C6 2.12 mm to (11.6, 11.7)
- moved L2 1.66 mm to (0.29, 9.01)
- moved L3 1.61 mm to (0.25, 7.55)
- moved U3 0.94 mm to (9.50, 3.25), flipped to the top
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Connections:
- new net CI: U$2.5, U1.AL13
- new net DI: U$2.6, U1.AL9
- net 3.3V: now also U$2.3
- net GND: now also U$2.4
Routing:
- net N$8: track 27.1 -> 11.4 mm
- net GND: track 95.8 -> 110.9 mm, vias 6 -> 7
- net OS: track 39.4 -> 26.7 mm, vias 5 -> 2
- net CI: track 0.00 -> 12.5 mm, vias 0 -> 1
- net N$9: track 10.8 -> 2.94 mm
- net 3.3V: track 112.1 -> 105.8 mm, vias 5 -> 7
- net SCL: track 17.7 -> 23.6 mm, vias 3 -> 2
- net DI: track 0.00 -> 4.26 mm, vias 0 -> 1
- net INT: track 17.1 -> 13.5 mm, vias 1 -> 2
- net N$2: track 7.80 -> 6.13 mm
- net N$14: track 2.74 -> 1.74 mm
- net N$7: track 2.05 -> 2.68 mm
- net SDA: vias 2 -> 1

Commit message: u
Parts:
- removed SW2: (no value), graftel-internal-ic:MICROBUILDER_BTN_EVQPQ_4.5MM
- added R5: 4.7K, Adafruit Circuit Playground Bluefruit:MICROBUILDER__0402MP
- added S1: KMR421GULCLFS, graftel-internal-ic:SW_KMR421GULCLFS
- R4: value (none) -> 4.7K
- moved J7 1.09 mm to (14.2, 6.28)
- moved J8 0.89 mm to (13.4, 4.96)
- moved J10 0.31 mm to (10.7, 17.0)
- moved J11 0.10 mm to (11.9, 16.0)
Connections:
- new net SW: R5.2, S1.2, S1.3, U1.AL15
- net 3.3V: now also S1.1, S1.4
- net GND: now also R5.1, S1.5
Routing:
- net GND: track 110.9 -> 0.00 mm, vias 7 -> 0
- net 3.3V: track 105.8 -> 0.00 mm, vias 7 -> 0
- net OS: track 26.7 -> 0.00 mm, vias 2 -> 0
- net SCL: track 23.6 -> 0.00 mm, vias 2 -> 0
- net SDA: track 23.2 -> 0.00 mm, vias 1 -> 0
- net INT: track 13.5 -> 0.00 mm, vias 2 -> 0
- net CI: track 12.5 -> 0.00 mm, vias 1 -> 0
- net N$8: track 11.4 -> 0.00 mm
- net 1.8V: track 9.20 -> 0.00 mm, vias 1 -> 0
- net N$1: track 6.14 -> 0.00 mm
- net N$2: track 6.13 -> 0.00 mm
- net N$3: track 5.88 -> 0.00 mm
- net DI: track 4.26 -> 0.00 mm, vias 1 -> 0
- net N$13: track 3.21 -> 0.00 mm
- net N$9: track 2.94 -> 0.00 mm
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- removed copper zone on layer 1, net GND
- removed copper zone on layer 16, net GND

Commit message: u
Parts:
- removed R5: 4.7K, Adafruit Circuit Playground Bluefruit:MICROBUILDER__0402MP
- moved R2 13.1 mm to (12.0, 7.36), flipped to the top, turned to 270 degrees
- moved R1 12.2 mm to (11.1, 7.38), flipped to the top, turned to 90 degrees
- moved C13 4.49 mm to (11.8, 3.47)
- moved C12 2.72 mm to (7.04, 3.28), turned to 270 degrees
- moved J8 0.92 mm to (13.8, 5.77)
- moved J7 0.79 mm to (14.5, 7.02)
- moved X1 0.47 mm to (2.28, 15.1)
- moved J9 0.34 mm to (12.8, 15.1)
- moved R4 0.33 mm to (-0.78, 5.10), flipped to the top, turned to 180 degrees
- moved R3 0.32 mm to (-0.78, 6.05), flipped to the top, turned to 0 degrees
- moved U$2 0.23 mm to (11.3, 4.52)
- moved C11 0.22 mm to (-0.24, 3.56)
- moved J10 0.16 mm to (10.9, 17.1)
- moved U3 0.15 mm to (9.35, 3.27), turned to 270 degrees
- moved J11 0.10 mm to (12.0, 16.1)
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Connections:
- net 3.3V: no longer S1.1, S1.4
- net GND: now also S1.2, S1.3; no longer R5.1
- net SW: now also S1.1, S1.4; no longer R5.2, S1.2, S1.3
Routing:
- net GND: track 0.00 -> 119.6 mm, vias 0 -> 3
- net 3.3V: track 0.00 -> 116.3 mm, vias 0 -> 8
- net OS: track 0.00 -> 25.2 mm, vias 0 -> 4
- net SCL: track 0.00 -> 22.8 mm
- net INT: track 0.00 -> 14.4 mm
- net SW: track 0.00 -> 10.9 mm, vias 0 -> 1
- net SDA: track 0.00 -> 10.4 mm, vias 0 -> 2
- net 1.8V: track 0.00 -> 10.2 mm, vias 0 -> 2
- net N$2: track 0.00 -> 7.65 mm
- net N$8: track 0.00 -> 7.27 mm, vias 0 -> 2
- net N$3: track 0.00 -> 6.40 mm
- net N$1: track 0.00 -> 6.29 mm
- net CI: track 0.00 -> 6.16 mm, vias 0 -> 1
- net DI: track 0.00 -> 4.44 mm, vias 0 -> 1
- net N$13: track 0.00 -> 3.32 mm
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
Commit message: u
Routing:
- net GND: track 119.6 -> 119.1 mm, vias 3 -> 7
- added copper zone on layer 1, net GND
- added copper zone on layer 16, net GND

Commit message: u
Connections:
- removed net N$14: C13.2, U3.8
- net 1_8V_EN: now also U1.AL19
- net 3.3V: now also U3.8
- net GND: now also C13.2
Routing:
- net 1_8V_EN: track 0.00 -> 11.2 mm, vias 0 -> 3
- net GND: track 119.1 -> 112.3 mm, vias 7 -> 9
- net N$14: track 2.87 -> 0.00 mm
- net 3.3V: track 116.5 -> 119.1 mm
- net N$2: track 7.65 -> 6.44 mm

Commit message: u
Parts:
- added U5: MAX32664GTGA+, graftel-internal-ic:21-100264_90-100089_MXM
- C3: value 1.0uF -> 1uF
Connections:
- new net EPAD: U5.25
- new net VCORE: U5.12
- new net VDD: U5.22
- new net VDD_2: U5.11
- new net VSS: U5.10
- new net VSS_2: U5.7
Changed lines of the file:
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@@
 <?xml version="1.0" encoding="utf-8"?>
 <!DOCTYPE eagle SYSTEM "eagle.dtd">
-<eagle version="9.5.2">
+<eagle version="9.6.2">
 <drawing>
 <settings>
@@
 <attribute name="VALUE" x="1.163603125" y="15.2677" size="0.6096" layer="27" rot="R180"/>
 </element>
-<element name="C3" library="Adafruit Circuit Playground Bluefruit" package="MICROBUILDER__0402MP" package3d_urn="urn:adsk.eagle:package:27347952/3" value="1.0uF" x="-1.3212" y="9.7742" smashed="yes" rot="R270">
+<element name="C3" library="Adafruit Circuit Playground Bluefruit" package="MICROBUILDER__0402MP" package3d_urn="urn:adsk.eagle:package:27347952/3" value="1uF" x="-1.3212" y="9.7742" smashed="yes" rot="R270">
 <attribute name="NAME" x="-0.6227" y="10.6632" size="0.6096" layer="25" rot="R270"/>
 <attribute name="VALUE" x="-2.5912" y="10.8537" size="0.6096" layer="27" rot="R270"/>
@@
 <attribute name="PACKAGE" value="None" x="6.9088" y="3.4798" size="1.778" layer="28" rot="MR0" display="off"/>
 <attribute name="PURCHASE-URL" value="https://pricing.snapeda.com/search/part/KMR421GULCLFS/?ref=eda" x="6.9088" y="3.4798" size="1.778" layer="28" rot="MR0" display="off"/>
+</element>
+<element name="U5" library="graftel-internal-ic" package="21-100264_90-100089_MXM" value="MAX32664GTGA+" x="-1.9558" y="-27.2796" smashed="yes">
+<attribute name="BUILT_BY" value="EMA_Rebekah" x="-1.9558" y="-27.2796" size="1.778" layer="27" display="off"/>
+<attribute name="COPYRIGHT" value="Copyright (C) 2018 Accelerated Designs. All rights reserved" x="-1.9558" y="-27.2796" size="1.778" layer="27" display="off"/>
+<attribute name="MANUFACTURER_PART_NUMBER" value="MAX32664GTGA+" x="-1.9558" y="-27.2796" size="1.778" layer="27" display="off"/>
+<attribute name="NAME" x="-5.2324" y="-27.9146" size="1.27" layer="25" ratio="6" rot="SR0"/>
+<attribute name="REVISION" value="2" x="-1.9558" y="-27.2796" size="1.778" layer="27" display="off"/>
+<attribute name="SOURCELIBRARY" value="Maxim_2020-02-10" x="-1.9558" y="-27.2796" size="1.778" layer="27" display="off"/>
+<attribute name="VALUE" x="-3.683" y="-27.9146" size="1.27" layer="21" ratio="6" rot="SR0"/>
+<attribute name="VENDOR" value="Maxim Integrated Products" x="-1.9558" y="-27.2796" size="1.778" layer="27" display="off"/>
 </element>
 </elements>
@@
 <wire x1="9.4742" y1="4.7752" x2="9.017" y2="4.318" width="0.127" layer="16"/>
 </signal>
+<signal name="VSS_2">
+<contactref element="U5" pad="7"/>
+</signal>
+<signal name="VSS">
+<contactref element="U5" pad="10"/>
+</signal>
+<signal name="VDD_2">
+<contactref element="U5" pad="11"/>
+</signal>
+<signal name="VCORE">
+<contactref element="U5" pad="12"/>
+</signal>
+<signal name="VDD">
+<contactref element="U5" pad="22"/>
+</signal>
+<signal name="EPAD">
+<contactref element="U5" pad="25"/>
+</signal>
 </signals>

Commit message: o
Connections:
- net N$1 renamed SWDIO
- net N$2 renamed SWCLK
- net N$3 renamed RESET
Changed lines of the file:
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@@
 <via x="-2.6416" y="6.477" extent="1-16" drill="0.3048"/>
 </signal>
-<signal name="N$1">
+<signal name="SWDIO">
 <contactref element="U1" pad="AA31"/>
 <contactref element="J11" pad="P$1"/>
@@
 <wire x1="11.938" y1="15.0114" x2="11.938" y2="16.002" width="0.127" layer="1"/>
 </signal>
-<signal name="N$2">
+<signal name="SWCLK">
 <contactref element="U1" pad="W31"/>
 <contactref element="J10" pad="P$1"/>
@@
 <wire x1="6.693" y1="13.33950625" x2="9.40629375" y2="16.0528" width="0.127" layer="1"/>
 </signal>
-<signal name="N$3">
+<signal name="RESET">
 <contactref element="U1" pad="AC31"/>
 <contactref element="J9" pad="P$1"/>
