File: PCB/sch/Baby_Mon_V0/baby_monitor_v0.sch (EAGLE design)
At the start: 37 parts, among them J1 BATT-COIN1CR1216, U1 NRF5340-QKAA-AB0-R, U2 MAX30101EFD+, U3 MAX30205MTA+, X1 XRCGB32M000F2P10R0

Commit message: u
Parts:
- added SW2: (no value), graftel-internal-ic:MICROBUILDER_SWITCH_TACT_SMTEVQPQ
- added U$2: (no value), graftel-internal-ic:MICROBUILDER_APA1022020
Connections:
- new net CI: U$2.CKI, U1G$3.P0.19
- new net DI: U$2.DI, U1G$3.P0.16/QPSI_[3]
- net 3.3V: now also U$2.VDD
- net GND: now also U$2.GND
Changed lines of the file:
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@@
 <part name="SUPPLY8" library="SparkFun-Aesthetics" deviceset="3.3V" device=""/>
 <part name="R4" library="Adafruit Circuit Playground Bluefruit" deviceset="MICROBUILDER_RESISTOR" device="_0402MP" override_package3d_urn="urn:adsk.eagle:package:27347952/2" override_package_urn="urn:adsk.eagle:footprint:27347953/1"/>
+<part name="U$2" library="graftel-internal-ic" deviceset="MICROBUILDER_APA102" device="2020"/>
+<part name="SUPPLY9" library="SparkFun-Aesthetics" deviceset="3.3V" device=""/>
+<part name="GND14" library="SparkFun-Aesthetics" deviceset="GND" device=""/>
+<part name="SW2" library="graftel-internal-ic" deviceset="MICROBUILDER_SWITCH_TACT_SMT" device="EVQPQ"/>
 </parts>
 <sheets>
@@
 <attribute name="VALUE" x="17.78" y="111.76" size="1.016" layer="96" font="vector" ratio="15" align="center"/>
 </instance>
+<instance part="U$2" gate="G$1" x="187.96" y="154.94" smashed="yes">
+<attribute name="NAME" x="177.8" y="166.116" size="1.27" layer="95"/>
+<attribute name="VALUE" x="177.8" y="142.24" size="1.27" layer="96"/>
+</instance>
+<instance part="SUPPLY9" gate="G$1" x="193.04" y="175.26" smashed="yes">
+<attribute name="VALUE" x="192.024" y="178.816" size="1.778" layer="96"/>
+</instance>
+<instance part="GND14" gate="1" x="187.96" y="134.62" smashed="yes">
+<attribute name="VALUE" x="185.42" y="132.08" size="1.778" layer="96"/>
+</instance>
+<instance part="SW2" gate="G$1" x="134.62" y="149.86" smashed="yes">
+<attribute name="NAME" x="132.08" y="156.21" size="1.27" layer="95"/>
+<attribute name="VALUE" x="132.08" y="144.78" size="1.27" layer="96"/>
+</instance>
 </instances>
 <busses>
@@
 <pinref part="C13" gate="G$1" pin="1"/>
 <wire x1="27.94" y1="149.86" x2="33.02" y2="149.86" width="0.1524" layer="91"/>
+</segment>
+<segment>
+<pinref part="SUPPLY9" gate="G$1" pin="3.3V"/>
+<pinref part="U$2" gate="G$1" pin="VDD"/>
+<wire x1="193.04" y1="175.26" x2="193.04" y2="167.64" width="0.1524" layer="91"/>
 </segment>
 </net>
@@
 <wire x1="15.24" y1="129.54" x2="15.24" y2="119.38" width="0.1524" layer="91"/>
 </segment>
+<segment>
+<pinref part="U$2" gate="G$1" pin="GND"/>
+<pinref part="GND14" gate="1" pin="GND"/>
+<wire x1="187.96" y1="142.24" x2="187.96" y2="137.16" width="0.1524" layer="91"/>
+</segment>
 </net>
 <net name="1.8V" class="0">
@@
 </segment>
 </net>
+<net name="DI" class="0">
+<segment>
+<pinref part="U1" gate="G$3" pin="P0.16/QPSI_[3]"/>
+<wire x1="88.9" y1="106.68" x2="76.2" y2="106.68" width="0.1524" layer="91"/>
+<label x="78.74" y="106.68" size="1.778" layer="95"/>
+</segment>
+<segment>
+<pinref part="U$2" gate="G$1" pin="DI"/>
+<wire x1="175.26" y1="149.86" x2="157.48" y2="149.86" width="0.1524" layer="91"/>
+<label x="165.1" y="149.86" size="1.778" layer="95"/>
+</segment>
+</net>
+<net name="CI" class="0">
+<segment>
+<pinref part="U1" gate="G$3" pin="P0.19"/>
+<wire x1="88.9" y1="99.06" x2="76.2" y2="99.06" width="0.1524" layer="91"/>
+<label x="78.74" y="99.06" size="1.778" layer="95"/>
+</segment>
+<segment>
+<pinref part="U$2" gate="G$1" pin="CKI"/>
+<wire x1="175.26" y1="147.32" x2="157.48" y2="147.32" width="0.1524" layer="91"/>
+<label x="165.1" y="147.32" size="1.778" layer="95"/>
+</segment>
+</net>

Commit message: u
Parts:
- removed SW2: (no value), graftel-internal-ic:MICROBUILDER_SWITCH_TACT_SMTEVQPQ
- added R5: 4.7K, Adafruit Circuit Playground Bluefruit:MICROBUILDER_RESISTOR_0402MP
- added S1: KMR421GULCLFS, graftel-internal-ic:KMR421GULCLFS
- R4: value (none) -> 4.7K
Connections:
- new net SW: R5.2, S1.2, S1.3, U1G$3.P0.21
- net 3.3V: now also S1.1, S1.4
- net GND: now also R5.1, S1.G

Commit message: u
Parts:
- removed R5: 4.7K, Adafruit Circuit Playground Bluefruit:MICROBUILDER_RESISTOR_0402MP
Connections:
- net 3.3V: no longer S1.1, S1.4
- net GND: now also S1.2, S1.3; no longer R5.1
- net SW: now also S1.1, S1.4; no longer R5.2, S1.2, S1.3

Commit message: u
Connections:
- removed net N$14: C13.2, U3.VDD
- net 1_8V_EN: now also U1G$2.P1.04
- net 3.3V: now also U3.VDD
- net GND: now also C13.2
Other:
- moved on the sheet: C13
Changed lines of the file:
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@@
 <?xml version="1.0" encoding="utf-8"?>
 <!DOCTYPE eagle SYSTEM "eagle.dtd">
-<eagle version="9.6.2">
+<eagle version="9.5.2">
 <drawing>
 <settings>
@@
 <attribute name="VALUE" x="58.42" y="119.38" size="1.778" layer="96"/>
 </instance>
-<instance part="C13" gate="G$1" x="38.1" y="149.86" smashed="yes" rot="R90">
-<attribute name="NAME" x="36.85" y="147.57" size="1.27" layer="95" font="vector" rot="R180" align="center"/>
-<attribute name="VALUE" x="36.85" y="152.16" size="1.27" layer="96" font="vector" rot="R180" align="center"/>
-</instance>
-<instance part="SUPPLY8" gate="G$1" x="27.94" y="152.4" smashed="yes">
-<attribute name="VALUE" x="26.924" y="155.956" size="1.778" layer="96"/>
+<instance part="C13" gate="G$1" x="71.12" y="134.62" smashed="yes">
+<attribute name="NAME" x="68.83" y="135.87" size="1.27" layer="95" font="vector" rot="R90" align="center"/>
+<attribute name="VALUE" x="73.42" y="135.87" size="1.27" layer="96" font="vector" rot="R90" align="center"/>
+</instance>
+<instance part="SUPPLY8" gate="G$1" x="71.12" y="142.24" smashed="yes">
+<attribute name="VALUE" x="70.104" y="145.796" size="1.778" layer="96"/>
 </instance>
 <instance part="R4" gate="G$1" x="17.78" y="111.76" smashed="yes">
@@
 </segment>
 <segment>
-<pinref part="SUPPLY8" gate="G$1" pin="3.3V"/>
-<wire x1="27.94" y1="152.4" x2="27.94" y2="149.86" width="0.1524" layer="91"/>
-<pinref part="C13" gate="G$1" pin="1"/>
-<wire x1="27.94" y1="149.86" x2="33.02" y2="149.86" width="0.1524" layer="91"/>
-</segment>
-<segment>
 <pinref part="SUPPLY9" gate="G$1" pin="3.3V"/>
 <pinref part="U$2" gate="G$1" pin="VDD"/>
 <wire x1="193.04" y1="175.26" x2="193.04" y2="167.64" width="0.1524" layer="91"/>
+</segment>
+<segment>
+<pinref part="U3" gate="A" pin="VDD"/>
+<wire x1="55.88" y1="134.62" x2="60.96" y2="134.62" width="0.1524" layer="91"/>
+<wire x1="60.96" y1="134.62" x2="60.96" y2="139.7" width="0.1524" layer="91"/>
+<pinref part="C13" gate="G$1" pin="1"/>
+<wire x1="60.96" y1="139.7" x2="71.12" y2="139.7" width="0.1524" layer="91"/>
+<pinref part="SUPPLY8" gate="G$1" pin="3.3V"/>
+<wire x1="71.12" y1="142.24" x2="71.12" y2="139.7" width="0.1524" layer="91"/>
+<junction x="71.12" y="139.7"/>
 </segment>
 </net>
@@
 <wire x1="66.04" y1="132.08" x2="60.96" y2="132.08" width="0.1524" layer="91"/>
 <junction x="60.96" y="132.08"/>
+<pinref part="C13" gate="G$1" pin="2"/>
+<wire x1="71.12" y1="132.08" x2="71.12" y2="127" width="0.1524" layer="91"/>
+<wire x1="71.12" y1="127" x2="60.96" y2="127" width="0.1524" layer="91"/>
 </segment>
 <segment>
@@
 <label x="17.78" y="165.1" size="1.778" layer="95"/>
 </segment>
+<segment>
+<pinref part="U1" gate="G$2" pin="P1.04"/>
+<wire x1="152.4" y1="114.3" x2="139.7" y2="114.3" width="0.1524" layer="91"/>
+<label x="139.7" y="114.3" size="1.778" layer="95"/>
+</segment>
 </net>
 <net name="SCL" class="0">
@@
 </segment>
 </net>
-<net name="N$14" class="0">
-<segment>
-<pinref part="C13" gate="G$1" pin="2"/>
-<wire x1="40.64" y1="149.86" x2="60.96" y2="149.86" width="0.1524" layer="91"/>
-<wire x1="60.96" y1="149.86" x2="60.96" y2="134.62" width="0.1524" layer="91"/>
-<pinref part="U3" gate="A" pin="VDD"/>
-<wire x1="60.96" y1="134.62" x2="55.88" y2="134.62" width="0.1524" layer="91"/>
-</segment>
-</net>

Commit message: u
Parts:
- added U5: MAX32664GTGA+, graftel-internal-ic:MAX32664GTGA+
- C3: value 1.0uF -> 1uF
Changed lines of the file:
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@@
 <?xml version="1.0" encoding="utf-8"?>
 <!DOCTYPE eagle SYSTEM "eagle.dtd">
-<eagle version="9.5.2">
+<eagle version="9.6.2">
 <drawing>
 <settings>
@@
 <part name="C1" library="Adafruit Circuit Playground Bluefruit" deviceset="MICROBUILDER_CAP_CERAMIC" device="_0402MP" package3d_urn="urn:adsk.eagle:package:27347952/3" value="1uF"/>
 <part name="C2" library="Adafruit Circuit Playground Bluefruit" deviceset="MICROBUILDER_CAP_CERAMIC" device="_0402MP" package3d_urn="urn:adsk.eagle:package:27347952/3" override_package3d_urn="urn:adsk.eagle:package:27369007/2" override_package_urn="urn:adsk.eagle:footprint:27369008/1" override_locally_modified="yes" value="1uF"/>
-<part name="C3" library="Adafruit Circuit Playground Bluefruit" deviceset="MICROBUILDER_CAP_CERAMIC" device="_0402MP" package3d_urn="urn:adsk.eagle:package:27347952/3" value="1.0uF"/>
+<part name="C3" library="Adafruit Circuit Playground Bluefruit" deviceset="MICROBUILDER_CAP_CERAMIC" device="_0402MP" package3d_urn="urn:adsk.eagle:package:27347952/3" value="1uF"/>
 <part name="C4" library="Adafruit Circuit Playground Bluefruit" deviceset="MICROBUILDER_CAP_CERAMIC" device="_0402MP" package3d_urn="urn:adsk.eagle:package:27347952/3" value="0.1uF"/>
 <part name="C5" library="Adafruit Circuit Playground Bluefruit" deviceset="MICROBUILDER_CAP_CERAMIC" device="_0402MP" package3d_urn="urn:adsk.eagle:package:27347952/3" value="0.1uF"/>
@@
 <part name="S1" library="graftel-internal-ic" deviceset="KMR421GULCLFS" device="" override_package3d_urn="urn:adsk.eagle:package:27368902/2" override_package_urn="urn:adsk.eagle:footprint:27368903/1"/>
 <part name="GND15" library="SparkFun-Aesthetics" deviceset="GND" device=""/>
+<part name="U5" library="graftel-internal-ic" deviceset="MAX32664GTGA+" device=""/>
 </parts>
 <sheets>
@@
 <attribute name="VALUE" x="144.78" y="137.16" size="1.778" layer="96"/>
 </instance>
+<instance part="U5" gate="A" x="35.56" y="45.72" smashed="yes">
+<attribute name="NAME" x="58.7756" y="54.8386" size="2.0828" layer="95" ratio="6" rot="SR0"/>
+<attribute name="VALUE" x="58.1406" y="52.2986" size="2.0828" layer="96" ratio="6" rot="SR0"/>
+</instance>
 </instances>

Commit message: o
Connections:
- net N$1 renamed SWDIO
- net N$2 renamed SWCLK
- net N$3 renamed RESET
Changed lines of the file:
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@@
 </busses>
 <nets>
-<net name="N$1" class="0">
+<net name="SWDIO" class="0">
 <segment>
 <pinref part="U1" gate="G$4" pin="SWDIO"/>
@@
 </segment>
 </net>
-<net name="N$2" class="0">
+<net name="SWCLK" class="0">
 <segment>
 <pinref part="U1" gate="G$4" pin="SWDCLK"/>
@@
 </segment>
 </net>
-<net name="N$3" class="0">
+<net name="RESET" class="0">
 <segment>
 <pinref part="U1" gate="G$4" pin="!RESET"/>
