File: PCB/sch/Baby_Mon_V0/baby_monitor_v2.brd (EAGLE design)
At the start: 25 x 25 mm, 29 parts, among them J1 BATT-COIN1CR1216, U2 MAX30101EFD+, U5 MAX32664GTGA+, Y1 CRYSTAL_OSCILLATOR0.126X0.061

Commit message: u
Parts:
- removed FRAME1, FRAME3: FRAME-LETTERNO_PACKAGE, SparkFun-Aesthetics:DUMMY
- added C1, C2: 22pF, Adafruit Circuit Playground Bluefruit:MICROBUILDER__0402MP
- added J8, J9: (no value), graftel-internal-ic:1X01_SMD_TINY_EXT
- added Y2: CRYSTAL_OSCILLATOR0.126X0.061, graftel-internal-ic:QUARTZ
- moved J6 51.7 mm to (15.2, 15.6)
- moved J5 51.6 mm to (13.0, 18.3)
- moved J4 49.2 mm to (14.1, 17.0)
- moved J7 47.8 mm to (17.0, 8.28)
- moved J3 39.1 mm to (16.6, 5.54)
- moved J2 14.0 mm to (15.6, 3.33)
Connections:
- new net N$1: C1.2, MDBT1.17, Y2.2
- new net N$2: MDBT1.22
- new net N$3: C2.2, MDBT1.18, Y2.1
- new net RXD: J8.P$1, MDBT1.48
- new net SWO: J7.P$1, MDBT1.47
- new net TXD: J9.P$1, MDBT1.49
- net 1_8V_EN: now also MDBT1.19
- net 3.3V: now also J2.P$1
- net CI: now also MDBT1.36
- net DI: now also MDBT1.37
- net GND: now also C1.1, C2.1, J3.P$1
- net MFIO: now also MDBT1.25
- net RESET: now also J6.P$1
- net RST: now also MDBT1.23
- net SWCLK: now also J5.P$1
- net SWDIO: now also J4.P$1
Routing:
- net GND: track 0.77 -> 132.7 mm, vias 1 -> 4
- net 3.3V: track 54.4 -> 75.4 mm, vias 3 -> 2
- net SWO: track 0.00 -> 14.9 mm, vias 0 -> 1
- net RXD: track 0.00 -> 13.6 mm, vias 0 -> 2
- net N$3: track 0.00 -> 12.7 mm
- net TXD: track 0.00 -> 12.0 mm
- net 1.8V: track 57.0 -> 46.4 mm
- net N$1: track 0.00 -> 9.51 mm
- net RESET: track 0.00 -> 9.11 mm, vias 0 -> 2
- net RST: track 1.79 -> 8.83 mm
- net MFIO: track 1.87 -> 7.78 mm, vias 0 -> 2
- net 1_8V_EN: track 0.00 -> 4.24 mm, vias 0 -> 1
- net SWDIO: track 0.00 -> 4.18 mm
- net CI: track 0.00 -> 4.14 mm, vias 0 -> 1
- net SWCLK: track 0.00 -> 3.22 mm
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- removed copper zone on layer 1, net GND
- removed copper zone on layer 16, net GND
