File: PCB/sch/Baby_Mon_V0/baby_monitor_v2.sch (EAGLE design)
At the start: 29 parts, among them J1 BATT-COIN1CR1216, U2 MAX30101EFD+, U5 MAX32664GTGA+, Y1 CRYSTAL_OSCILLATOR0.126X0.061

Commit message: u
Parts:
- removed FRAME1, FRAME3: FRAME-LETTERNO_PACKAGE, SparkFun-Aesthetics:FRAME-LETTERNO_PACKAGE
- added C1, C2: 22pF, Adafruit Circuit Playground Bluefruit:MICROBUILDER_CAP_CERAMIC_0402MP
- added J8, J9: (no value), graftel-internal-ic:M01TINY_SMD_EXT
- added Y2: CRYSTAL_OSCILLATOR0.126X0.061, graftel-internal-ic:CRYSTAL_OSCILLATOR0.126X0.061
Connections:
- new net N$1: C1.2, MDBT1.P0.00/XL1, Y2.2
- new net N$2: MDBT1.P0.06
- new net N$3: C2.2, MDBT1.P0.01/XL2, Y2.1
- new net RXD: J8.1, MDBT1.P0.24
- new net SWO: J7.1, MDBT1.P1.00
- new net TXD: J9.1, MDBT1.P0.25
- net 1_8V_EN: now also MDBT1.P0.26
- net 3.3V: now also J2.1
- net CI: now also MDBT1.P0.14
- net DI: now also MDBT1.P0.13
- net GND: now also C1.1, C2.1, J3.1
- net MFIO: now also MDBT1.P1.08
- net RESET: now also J6.1
- net RST: now also MDBT1.P0.07
- net SWCLK: now also J5.1
- net SWDIO: now also J4.1
