File: PCB/sch/Baby_Mon_V0/baby_monitor_v1.brd (EAGLE design)
At the start: 20 x 20 mm, 44 parts, among them J1 BATT-COIN1CR1216, U1 NRF5340-QKAA-AB0-R, U2 MAX30101EFD+, U5 MAX32664GTGA+, X1 XRCGB32M000F2P10R0, Y1 CRYSTAL_OSCILLATOR0.126X0.061

Commit message: u
Parts:
- moved R7 10.0 mm to (7.26, 1.19), turned to 270 degrees
- moved Y1 9.29 mm to (6.81, -1.38), turned to 180 degrees
- moved R6 9.14 mm to (7.26, 3.38), turned to 270 degrees
- moved R5 8.09 mm to (2.03, -0.58), turned to 0 degrees
- moved C14 6.05 mm to (13.6, 2.13), turned to 90 degrees
- moved R4 5.02 mm to (8.54, 4.93), turned to 180 degrees
- moved C10 4.66 mm to (-1.41, 3.06)
- moved R1 4.62 mm to (10.6, 4.94), turned to 0 degrees
- moved C11 4.50 mm to (-3.90, 6.18)
- moved U4 4.19 mm to (-1.18, 6.00)
- moved J8 3.17 mm to (15.8, 6.12)
- moved U$2 3.07 mm to (12.4, 7.39)
- moved R2 3.00 mm to (3.37, 5.13), turned to 180 degrees
- moved C1 2.56 mm to (-1.47, 9.10), turned to 180 degrees
- moved J7 2.55 mm to (16.6, 8.49)
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Routing:
- net GND: track 112.0 -> 146.6 mm, vias 5 -> 7
- net 3.3V: track 101.7 -> 132.6 mm, vias 6 -> 8
- net SCL: track 30.5 -> 6.04 mm, vias 2 -> 0
- net 1.8V: track 28.0 -> 45.7 mm, vias 1 -> 6
- net MFIO: track 0.00 -> 16.1 mm, vias 0 -> 6
- net RST: track 8.93 -> 22.6 mm, vias 0 -> 2
- net SEN_SDA: track 12.4 -> 22.0 mm
- net SW: track 12.1 -> 21.7 mm
- net HR_INT: track 12.2 -> 20.0 mm
- net SEN_SCL: track 9.33 -> 16.0 mm, vias 0 -> 2
- net N$8: track 12.5 -> 18.9 mm
- net N$9: track 12.2 -> 6.19 mm
- net SDA: track 0.00 -> 5.98 mm
- net N$15: track 0.00 -> 5.10 mm
- net 1_8V_EN: track 9.78 -> 13.6 mm
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Other:
- board size 20 x 20 mm -> 25 x 25 mm

Commit message: o
Parts:
- removed L2: 15nH, Adafruit Circuit Playground Bluefruit:NORDIC_MISC_RESC0402_N
- L1: value 15nH -> 10uH; device Adafruit Circuit Playground Bluefruit:NORDIC_MISC_RESC0402_N -> Adafruit Circuit Playground Bluefruit:NORDIC_MISC_RESC0603_N
- moved L1 40.1 mm to (-5.41, -28.2), turned to 0 degrees
Connections:
- removed net DCCH: U1.J1
- removed net N$6: L2.2, L3.1
- net 3.3V: now also L1.1
- net N$5: now also U1.J1; no longer L4.1
- net N$8: now also L4.1; no longer L1.1
- net N$9: now also L3.1; no longer L2.1
Routing:
- net N$9: track 6.19 -> 4.53 mm
- net N$6: track 1.49 -> 0.00 mm
- net N$5: track 1.35 -> 0.00 mm
- added copper zone on layer 1, net GND
- added copper zone on layer 16, net GND

Commit message: u
Parts:
- moved L1 35.8 mm to (2.79, 6.60)
Connections:
- removed net VDDH: U1.E1
- net 3.3V: now also U1.E1
Routing:
- net N$8: track 18.6 -> 23.8 mm
- net N$9: track 4.53 -> 8.07 mm
- net N$5: track 0.00 -> 2.61 mm
- net 3.3V: track 132.7 -> 130.8 mm, vias 8 -> 9
- net GND: track 146.7 -> 148.3 mm, vias 7 -> 9

Commit message: u
Connections:
- net N$1 renamed SWDIO
- net N$2 renamed SWDCLK
- net N$3 renamed RESET
Routing:
- net GND: track 148.3 -> 144.3 mm, vias 9 -> 11
- net SWDCLK: track 8.97 -> 7.42 mm
Changed lines of the file:
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@@
 <wire x1="12.573" y1="14.605" x2="12.51938125" y2="14.68691875" width="0.127" layer="1"/>
 <wire x1="12.573" y1="13.462" x2="12.53235625" y2="13.3524" width="0.127" layer="1"/>
-<wire x1="12.319" y1="17.653" x2="7.366" y2="17.653" width="0.127" layer="1"/>
-<wire x1="12.446" y1="17.526" x2="12.319" y2="17.653" width="0.127" layer="1"/>
-<wire x1="13.589" y1="17.526" x2="12.446" y2="17.526" width="0.127" layer="1"/>
-<wire x1="13.843" y1="17.78" x2="13.589" y2="17.526" width="0.127" layer="1"/>
-<wire x1="14.224" y1="17.78" x2="13.843" y2="17.78" width="0.127" layer="1"/>
-<wire x1="14.732" y1="17.272" x2="14.224" y2="17.78" width="0.127" layer="1"/>
-<wire x1="14.732" y1="16.383" x2="14.732" y2="17.272" width="0.127" layer="1"/>
-<wire x1="13.081" y1="14.732" x2="14.732" y2="16.383" width="0.127" layer="1"/>
-<wire x1="12.573" y1="14.732" x2="13.081" y2="14.732" width="0.127" layer="1"/>
-<wire x1="7.366" y1="17.653" x2="7.262" y2="17.7336" width="0.127" layer="1"/>
-<wire x1="12.573" y1="14.732" x2="12.51938125" y2="14.68691875" width="0.127" layer="1"/>
 <wire x1="14.859" y1="8.509" x2="16.51" y2="8.509" width="0.127" layer="1"/>
 <wire x1="12.573" y1="10.795" x2="14.859" y2="8.509" width="0.127" layer="1"/>
@@
 <wire x1="4.790440625" y1="7.7851" x2="4.790440625" y2="3.982759375" width="0.127" layer="1"/>
 <wire x1="4.790440625" y1="3.982759375" x2="5.3137" y2="3.4595" width="0.127" layer="1"/>
+<wire x1="7.262" y1="17.7336" x2="8.107" y2="17.7336" width="0.1524" layer="1"/>
+<wire x1="8.107" y1="17.7336" x2="8.128" y2="17.7546" width="0.1524" layer="1"/>
+<via x="8.128" y="17.7546" extent="1-16" drill="0.35"/>
+<wire x1="8.128" y1="17.7546" x2="10.6161" y2="17.7546" width="0.1524" layer="16"/>
+<wire x1="10.6161" y1="17.7546" x2="13.1064" y2="15.2643" width="0.1524" layer="16"/>
+<wire x1="13.1064" y1="15.2643" x2="13.0967625" y2="15.2643" width="0.1524" layer="1"/>
+<wire x1="13.0967625" y1="15.2643" x2="12.51938125" y2="14.68691875" width="0.1524" layer="1"/>
+<via x="13.1064" y="15.2643" extent="1-16" drill="0.35"/>
 </signal>
-<signal name="N$1">
+<signal name="SWDIO">
 <contactref element="U1" pad="AA31"/>
 <contactref element="J11" pad="P$1"/>
@@
 <wire x1="13.97" y1="17.018" x2="14.0338" y2="17.0354" width="0.127" layer="1"/>
 </signal>
-<signal name="N$2">
+<signal name="SWDCLK">
 <contactref element="U1" pad="W31"/>
 <contactref element="J10" pad="P$1"/>
-<wire x1="6.604" y1="16.256" x2="6.604" y2="15.24" width="0.127" layer="1"/>
-<wire x1="6.731" y1="16.383" x2="6.604" y2="16.256" width="0.127" layer="1"/>
-<wire x1="6.731" y1="18.034" x2="6.731" y2="16.383" width="0.127" layer="1"/>
-<wire x1="6.985" y1="18.288" x2="6.731" y2="18.034" width="0.127" layer="1"/>
-<wire x1="12.7" y1="18.288" x2="6.985" y2="18.288" width="0.127" layer="1"/>
-<wire x1="6.604" y1="15.24" x2="6.596" y2="15.1952" width="0.127" layer="1"/>
 <wire x1="12.7" y1="18.288" x2="12.705" y2="18.2846" width="0.127" layer="1"/>
+<wire x1="6.596" y1="15.1952" x2="6.6803" y2="15.2795" width="0.1524" layer="1"/>
+<wire x1="6.6803" y1="15.2795" x2="6.6803" y2="15.32596875" width="0.1524" layer="1"/>
+<wire x1="6.6803" y1="15.32596875" x2="6.79433125" y2="15.44" width="0.1524" layer="1"/>
+<wire x1="6.79433125" y1="15.44" x2="6.814115625" y2="15.4726625" width="0.1524" layer="1"/>
+<wire x1="6.814115625" y1="15.4726625" x2="6.831184375" y2="15.476853125" width="0.1524" layer="1"/>
+<wire x1="6.831184375" y1="15.476853125" x2="6.86523125" y2="15.5109" width="0.1524" layer="1"/>
+<wire x1="6.86523125" y1="15.5109" x2="6.878725" y2="15.5109" width="0.1524" layer="1"/>
+<wire x1="6.878725" y1="15.5109" x2="9.655825" y2="18.288" width="0.1524" layer="1"/>
+<wire x1="9.655825" y1="18.288" x2="12.7" y2="18.288" width="0.1524" layer="1"/>
 </signal>
-<signal name="N$3">
+<signal name="RESET">
 <contactref element="U1" pad="AC31"/>
 <contactref element="J9" pad="P$1"/>

Commit message: u
Parts:
- removed FRAME3: FRAME-LETTERNO_PACKAGE, SparkFun-Aesthetics:DUMMY
Changed lines of the file:
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@@
 <attribute name="VERSION" value="v01" x="-1.016" y="-23.368" size="1.778" layer="27" display="off"/>
-</element>
-<element name="FRAME3" library="SparkFun-Aesthetics" package="DUMMY" value="FRAME-LETTERNO_PACKAGE" x="-2.032" y="-24.384" smashed="yes">
-<attribute name="DESIGNER" value="Nobody" x="-2.032" y="-24.384" size="1.778" layer="27" display="off"/>
-<attribute name="VERSION" value="v01" x="-2.032" y="-24.384" size="1.778" layer="27" display="off"/>
 </element>
 <element name="J7" library="graftel-internal-ic" package="1X01_TINY" value="" x="16.6158" y="8.4896" smashed="yes"/>
