File: PCB/sch/Baby_Mon_V0/baby_monitor_v1.sch (EAGLE design)
At the start: 44 parts, among them J1 BATT-COIN1CR1216, U1 NRF5340-QKAA-AB0-R, U2 MAX30101EFD+, U5 MAX32664GTGA+, X1 XRCGB32M000F2P10R0, Y1 CRYSTAL_OSCILLATOR0.126X0.061

Commit message: o
Parts:
- removed L2: 15nH, Adafruit Circuit Playground Bluefruit:NORDIC_MISC_INDUCTOR_0402_N
- L1: value 15nH -> 10uH; device Adafruit Circuit Playground Bluefruit:NORDIC_MISC_INDUCTOR_0402_N -> Adafruit Circuit Playground Bluefruit:NORDIC_MISC_INDUCTOR_0603_N
Connections:
- removed net N$6: L2.2, L3.1
- net 3.3V: now also L1.1
- net N$5: now also U1G$1.DCCH; no longer L4.1
- net N$8: now also L4.1; no longer L1.1
- net N$9: now also L3.1; no longer L2.1
Other:
- moved on the sheet: L1
Changed lines of the file:
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@@
 <part name="J10" library="graftel-internal-ic" deviceset="M01" device="TINY"/>
 <part name="J11" library="graftel-internal-ic" deviceset="M01" device="TINY"/>
-<part name="L1" library="Adafruit Circuit Playground Bluefruit" deviceset="NORDIC_MISC_INDUCTOR" device="_0402_N" value="15nH"/>
-<part name="L2" library="Adafruit Circuit Playground Bluefruit" deviceset="NORDIC_MISC_INDUCTOR" device="_0402_N" value="15nH"/>
 <part name="L3" library="Adafruit Circuit Playground Bluefruit" deviceset="NORDIC_MISC_INDUCTOR" device="_0603_N" value="10uH"/>
 <part name="L4" library="Adafruit Circuit Playground Bluefruit" deviceset="NORDIC_MISC_INDUCTOR" device="_0603_N" value="10uH"/>
@@
 <part name="S1" library="graftel-internal-ic" deviceset="KMR421GULCLFS" device="" override_package3d_urn="urn:adsk.eagle:package:27368902/2" override_package_urn="urn:adsk.eagle:footprint:27368903/1"/>
 <part name="GND15" library="SparkFun-Aesthetics" deviceset="GND" device=""/>
-<part name="U5" library="graftel-internal-ic" deviceset="MAX32664GTGA+" device=""/>
+<part name="U5" library="graftel-internal-ic" deviceset="MAX32664GTGA+" device="" override_package3d_urn="urn:adsk.eagle:package:27725412/2" override_package_urn="urn:adsk.eagle:footprint:27725415/1"/>
 <part name="C14" library="Adafruit Circuit Playground Bluefruit" deviceset="MICROBUILDER_CAP_CERAMIC" device="_0402MP" package3d_urn="urn:adsk.eagle:package:27347952/3" override_package3d_urn="urn:adsk.eagle:package:27347947/2" override_package_urn="urn:adsk.eagle:footprint:27347948/1" override_locally_modified="yes" value="1uF"/>
 <part name="C15" library="Adafruit Circuit Playground Bluefruit" deviceset="MICROBUILDER_CAP_CERAMIC" device="_0402MP" package3d_urn="urn:adsk.eagle:package:27347952/3" override_package3d_urn="urn:adsk.eagle:package:27347947/2" override_package_urn="urn:adsk.eagle:footprint:27347948/1" override_locally_modified="yes" value="1uF"/>
@@
 <part name="R7" library="Adafruit Circuit Playground Bluefruit" deviceset="MICROBUILDER_RESISTOR" device="_0402MP" package3d_urn="urn:adsk.eagle:package:27347952/3" value="4.7K"/>
 <part name="SUPPLY12" library="SparkFun-Aesthetics" deviceset="3.3V" device=""/>
+<part name="L1" library="Adafruit Circuit Playground Bluefruit" deviceset="NORDIC_MISC_INDUCTOR" device="_0603_N" value="10uH"/>
 </parts>
 <sheets>
@@
 <attribute name="DRAWING_NAME" x="162.814" y="17.78" size="2.7432" layer="94" font="vector"/>
 </instance>
-<instance part="L1" gate="L$1" x="43.18" y="76.2" smashed="yes" rot="R90">
-<attribute name="NAME" x="38.1" y="78.74" size="1.778" layer="95" rot="R90"/>
-<attribute name="VALUE" x="48.26" y="78.74" size="1.778" layer="96" rot="R90"/>
-</instance>
-<instance part="L2" gate="L$1" x="43.18" y="63.5" smashed="yes" rot="R90">
-<attribute name="NAME" x="38.1" y="66.04" size="1.778" layer="95" rot="R90"/>
-<attribute name="VALUE" x="48.26" y="66.04" size="1.778" layer="96" rot="R90"/>
-</instance>
 <instance part="L3" gate="L$1" x="63.5" y="63.5" smashed="yes" rot="R90">
 <attribute name="NAME" x="58.42" y="66.04" size="1.778" layer="95" rot="R90"/>
@@
 <instance part="GND5" gate="1" x="30.48" y="60.96" smashed="yes">
 <attribute name="VALUE" x="27.94" y="58.42" size="1.778" layer="96"/>
+</instance>
+<instance part="L1" gate="L$1" x="63.5" y="53.34" smashed="yes" rot="R90">
+<attribute name="NAME" x="58.42" y="55.88" size="1.778" layer="95" rot="R90"/>
+<attribute name="VALUE" x="68.58" y="55.88" size="1.778" layer="96" rot="R90"/>
 </instance>
 </instances>
@@
 <wire x1="60.96" y1="45.72" x2="55.88" y2="45.72" width="0.1524" layer="91"/>
 <junction x="60.96" y="55.88"/>
-<wire x1="60.96" y1="55.88" x2="50.8" y2="55.88" width="0.1524" layer="91"/>
+<wire x1="60.96" y1="55.88" x2="55.88" y2="55.88" width="0.1524" layer="91"/>
 <pinref part="C3" gate="G$1" pin="1"/>
+<wire x1="55.88" y1="55.88" x2="50.8" y2="55.88" width="0.1524" layer="91"/>
 <wire x1="50.8" y1="55.88" x2="50.8" y2="45.72" width="0.1524" layer="91"/>
 <pinref part="C4" gate="G$1" pin="1"/>
@@
 <wire x1="124.46" y1="71.12" x2="137.16" y2="71.12" width="0.1524" layer="91"/>
 <junction x="124.46" y="71.12"/>
+<pinref part="L1" gate="L$1" pin="1"/>
+<wire x1="55.88" y1="53.34" x2="55.88" y2="55.88" width="0.1524" layer="91"/>
+<junction x="55.88" y="55.88"/>
 </segment>
 </net>
@@
 </segment>
 </net>
-<net name="N$5" class="0">
-<segment>
-<pinref part="L4" gate="L$1" pin="1"/>
-<pinref part="L1" gate="L$1" pin="2"/>
-<wire x1="55.88" y1="76.2" x2="50.8" y2="76.2" width="0.1524" layer="91"/>
-</segment>
-</net>
-<net name="N$6" class="0">
-<segment>
-<pinref part="L3" gate="L$1" pin="1"/>
-<pinref part="L2" gate="L$1" pin="2"/>
-<wire x1="55.88" y1="63.5" x2="50.8" y2="63.5" width="0.1524" layer="91"/>
-</segment>
-</net>
 <net name="N$7" class="0">
 <segment>
@@
 <net name="N$8" class="0">
 <segment>
-<pinref part="L1" gate="L$1" pin="1"/>
-<wire x1="35.56" y1="76.2" x2="30.48" y2="76.2" width="0.1524" layer="91"/>
 <pinref part="C2" gate="G$1" pin="1"/>
-<wire x1="30.48" y1="76.2" x2="30.48" y2="73.66" width="0.1524" layer="91"/>
 <pinref part="U1" gate="G$1" pin="DECR"/>
 <wire x1="30.48" y1="73.66" x2="35.56" y2="73.66" width="0.1524" layer="91"/>
-<junction x="30.48" y="73.66"/>
 <pinref part="U1" gate="G$1" pin="DECRF"/>
 <wire x1="35.56" y1="73.66" x2="76.2" y2="73.66" width="0.1524" layer="91"/>
@@
 <wire x1="35.56" y1="71.12" x2="35.56" y2="73.66" width="0.1524" layer="91"/>
 <junction x="35.56" y="73.66"/>
+<wire x1="30.48" y1="73.66" x2="30.48" y2="76.2" width="0.1524" layer="91"/>
+<junction x="30.48" y="73.66"/>
+<pinref part="L4" gate="L$1" pin="1"/>
+<wire x1="30.48" y1="76.2" x2="55.88" y2="76.2" width="0.1524" layer="91"/>
 </segment>
 </net>
 <net name="N$9" class="0">
 <segment>
-<pinref part="L2" gate="L$1" pin="1"/>
-<wire x1="35.56" y1="63.5" x2="35.56" y2="60.96" width="0.1524" layer="91"/>
-<pinref part="C1" gate="G$1" pin="1"/>
-<wire x1="35.56" y1="60.96" x2="35.56" y2="58.42" width="0.1524" layer="91"/>
-<wire x1="35.56" y1="58.42" x2="30.48" y2="58.42" width="0.1524" layer="91"/>
 <pinref part="U1" gate="G$1" pin="DECD"/>
 <wire x1="76.2" y1="60.96" x2="35.56" y2="60.96" width="0.1524" layer="91"/>
+<pinref part="C1" gate="G$1" pin="1"/>
+<wire x1="30.48" y1="58.42" x2="35.56" y2="58.42" width="0.1524" layer="91"/>
+<wire x1="35.56" y1="58.42" x2="35.56" y2="60.96" width="0.1524" layer="91"/>
+<pinref part="L3" gate="L$1" pin="1"/>
+<wire x1="35.56" y1="60.96" x2="35.56" y2="63.5" width="0.1524" layer="91"/>
+<wire x1="35.56" y1="63.5" x2="55.88" y2="63.5" width="0.1524" layer="91"/>
 <junction x="35.56" y="60.96"/>
 </segment>
 </net>
+<net name="N$5" class="0">
+<segment>
+<pinref part="U1" gate="G$1" pin="DCCH"/>
+<pinref part="L1" gate="L$1" pin="2"/>
+<wire x1="76.2" y1="53.34" x2="71.12" y2="53.34" width="0.1524" layer="91"/>
+</segment>
+</net>

Commit message: u
Connections:
- net 3.3V: now also U1G$1.VDDH
Changed lines of the file:
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@@
 <junction x="60.96" y="66.04"/>
 <pinref part="C7" gate="G$1" pin="1"/>
-<wire x1="60.96" y1="55.88" x2="60.96" y2="45.72" width="0.1524" layer="91"/>
+<wire x1="60.96" y1="55.88" x2="60.96" y2="50.8" width="0.1524" layer="91"/>
+<wire x1="60.96" y1="50.8" x2="60.96" y2="45.72" width="0.1524" layer="91"/>
 <wire x1="60.96" y1="45.72" x2="55.88" y2="45.72" width="0.1524" layer="91"/>
 <junction x="60.96" y="55.88"/>
@@
 <wire x1="55.88" y1="53.34" x2="55.88" y2="55.88" width="0.1524" layer="91"/>
 <junction x="55.88" y="55.88"/>
+<pinref part="U1" gate="G$1" pin="VDDH"/>
+<wire x1="76.2" y1="50.8" x2="60.96" y2="50.8" width="0.1524" layer="91"/>
+<junction x="60.96" y="50.8"/>
 </segment>
 </net>

Commit message: u
Connections:
- net N$1 renamed SWDIO
- net N$2 renamed SWDCLK
- net N$3 renamed RESET
Changed lines of the file:
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@@
 </busses>
 <nets>
-<net name="N$1" class="0">
+<net name="SWDIO" class="0">
 <segment>
 <pinref part="U1" gate="G$4" pin="SWDIO"/>
@@
 </segment>
 </net>
-<net name="N$2" class="0">
+<net name="SWDCLK" class="0">
 <segment>
 <pinref part="U1" gate="G$4" pin="SWDCLK"/>
@@
 </segment>
 </net>
-<net name="N$3" class="0">
+<net name="RESET" class="0">
 <segment>
 <pinref part="U1" gate="G$4" pin="!RESET"/>

Commit message: u
Parts:
- removed FRAME3: FRAME-LETTERNO_PACKAGE, SparkFun-Aesthetics:FRAME-LETTERNO_PACKAGE
